File: not-so-fullsize-ortho.kicad_pcb (KiCad board)
At the start: 2 copper layers, 340.4 x 81.3 mm, 153 parts, among them K0 Home, K1 Tab, K10 O, K11 P, K12 Back Space, K13 Delete, K14 1, K15 2, K16 3, K17 End, K18 Esc, K19 A, K2 Q, K20 S, K21 D, K22 F, K23 G, K24 H, K25 J, K26 K, K27 L, K28 ;, K29 ', K3 W, K30 Return, K31 4, K32 5, K33 6, K34 Vol +, K35 Shift, K36 Z, K37 X, K38 C, K39 V, K4 E, K40 B, K41 N, K42 M, K43 ,, K44 ., K45 /, K46 Shift, K47 7, K48 8, K49 9, K5 R, K50 &uarr;, K51 Vol -, K52 Ctrl, K53 Alt, K54 Super, K55 &dArr;, K56 Blank, K57 &uArr;, K58 Alt, K59 Fn, K6 T, K60 0, K61 Enter, K62 &larr;, K63 &darr;, K64 &rarr;, K7 Y, K8 U, K9 I, U1 Pico

Commit message: rework for rp2040 (not pico dev board)
kicad 8 version bump, much better schematic, some DRC rules, start with layout of rp2040/USB portion of board, will need to reroute all the rows/cols when done.
Parts:
- removed C3, C4: 0.1u, Capacitor_SMD:C_0805_2012Metric_Pad1.18x1.45mm_HandSolder
- removed C5: 4.7u, Capacitor_SMD:C_0805_2012Metric_Pad1.18x1.45mm_HandSolder
- removed D0: D, Diode_SMD:D_0805_2012Metric_Pad1.15x1.40mm_HandSolder
- removed K0: Home, Switch_Keyboard_Cherry_MX:SW_Cherry_MX_PCB_1.00u
- added C10: 100n, Capacitor_SMD:C_0402_1005Metric, F.Cu at (305.6, 67.5)
- added C11: 100n, Capacitor_SMD:C_0402_1005Metric, F.Cu at (305.6, 69.4)
- added C12: 100n, Capacitor_SMD:C_0402_1005Metric, F.Cu at (305.6, 71.4)
- added C13: 1u, Capacitor_SMD:C_0402_1005Metric, F.Cu at (308.4, 63.5)
- added C14: 100n, Capacitor_SMD:C_0402_1005Metric, F.Cu at (308.4, 65.5)
- added C15: 1u, Capacitor_SMD:C_0402_1005Metric, F.Cu at (308.4, 67.5)
- added C16: 100n, Capacitor_SMD:C_0402_1005Metric, F.Cu at (308.4, 69.4)
- added C17: 100n, Capacitor_SMD:C_0402_1005Metric, F.Cu at (308.4, 71.4)
- added C18: 100n, Capacitor_SMD:C_0402_1005Metric, F.Cu at (311.3, 63.5)
- added C19: 100n, Capacitor_SMD:C_0402_1005Metric, F.Cu at (311.3, 65.5)
- added C20: 100n, Capacitor_SMD:C_0402_1005Metric, F.Cu at (311.3, 67.5)
- added C21: 100n, Capacitor_SMD:C_0402_1005Metric, F.Cu at (311.3, 69.4)
- added C22: 10u, Capacitor_SMD:C_0805_2012Metric, F.Cu at (315.0, 71.2)
- added C6: 15p, Capacitor_SMD:C_0402_1005Metric, F.Cu at (305.6, 63.5)
- added C7: 15p, Capacitor_SMD:C_0402_1005Metric, B.Cu at (307.2, 92.5)
- added D65: D, Diode_SMD:D_0805_2012Metric_Pad1.15x1.40mm_HandSolder, B.Cu at (65.2, 85.8)
- added J1: Conn_01x02, Connector_PinHeader_2.54mm:PinHeader_1x02_P2.54mm_Vertical, F.Cu at (277.1, 68.8)
- added J2: USB_C_Receptacle_USB2.0_16P, Connector_USB:USB_C_Receptacle_HRO_TYPE-C-31-M-12, B.Cu at (318.0, 81.2)
- added J3: Conn_01x03, Connector_PinHeader_2.54mm:PinHeader_1x03_P2.54mm_Vertical, F.Cu at (304.0, 98.5)
- added K65: Enter, PCM_Switch_Keyboard_Hotswap_Kailh:SW_Hotswap_Kailh_MX_1.00u, F.Cu at (53.3, 88.9)
- added R1: 1k, Resistor_SMD:R_0402_1005Metric, F.Cu at (302.7, 63.5)
- added R2: DNF, Resistor_SMD:R_0402_1005Metric, F.Cu at (302.7, 65.5)
- added R3: 1k, Resistor_SMD:R_0402_1005Metric, B.Cu at (308.2, 91.0)
- added R4: 27, Resistor_SMD:R_0402_1005Metric, B.Cu at (323.8, 94.8)
- added R5: 27, Resistor_SMD:R_0402_1005Metric, B.Cu at (323.8, 93.5)
- added R6: 5.1k, Resistor_SMD:R_0402_1005Metric, B.Cu at (315.0, 87.0)
- added R7: 5.1k, Resistor_SMD:R_0402_1005Metric, B.Cu at (320.2, 87.0)
- added U2: NCP1117-3.3_SOT223, Package_TO_SOT_SMD:SOT-223-3_TabPin2, F.Cu at (317.5, 118.0)
- added U3: W25Q128JVS, Package_SO:SOIC-8_5.23x5.23mm_P1.27mm, B.Cu at (318.0, 104.0)
- added U5: RP2040, Package_DFN_QFN:QFN-56-1EP_7x7mm_P0.4mm_EP3.2x3.2mm, B.Cu at (318.4, 95.3)
- added Y1: ABM8-272-T3, Crystal:Crystal_SMD_3225-4Pin_3.2x2.5mm, B.Cu at (310.5, 94.0)
- C1, C2: value 0.1u -> 10u; footprint Capacitor_SMD:C_0805_2012Metric_Pad1.18x1.45mm_HandSolder -> Capacitor_SMD:C_0805_2012Metric
- H1, H2, H3, H4: footprint MountingHole:MountingHole_3.2mm_M3_DIN965 -> MountingHole:MountingHole_2.2mm_M2
- K1: value Tab -> Home; footprint Switch_Keyboard_Cherry_MX:SW_Cherry_MX_PCB_1.00u -> PCM_Switch_Keyboard_Hotswap_Kailh:SW_Hotswap_Kailh_MX_1.00u
- K10: value O -> A; footprint Switch_Keyboard_Cherry_MX:SW_Cherry_MX_PCB_1.00u -> PCM_Switch_Keyboard_Hotswap_Kailh:SW_Hotswap_Kailh_MX_1.00u
- K11: value P -> Z; footprint Switch_Keyboard_Cherry_MX:SW_Cherry_MX_PCB_1.00u -> PCM_Switch_Keyboard_Hotswap_Kailh:SW_Hotswap_Kailh_MX_1.00u
- K12: value Back Space -> Alt; footprint Switch_Keyboard_Cherry_MX:SW_Cherry_MX_PCB_1.00u -> PCM_Switch_Keyboard_Hotswap_Kailh:SW_Hotswap_Kailh_MX_1.00u
- K13: value Delete -> W; footprint Switch_Keyboard_Cherry_MX:SW_Cherry_MX_PCB_1.00u -> PCM_Switch_Keyboard_Hotswap_Kailh:SW_Hotswap_Kailh_MX_1.00u
- K14: value 1 -> S; footprint Switch_Keyboard_Cherry_MX:SW_Cherry_MX_PCB_1.00u -> PCM_Switch_Keyboard_Hotswap_Kailh:SW_Hotswap_Kailh_MX_1.00u
- K15: value 2 -> X; footprint Switch_Keyboard_Cherry_MX:SW_Cherry_MX_PCB_1.00u -> PCM_Switch_Keyboard_Hotswap_Kailh:SW_Hotswap_Kailh_MX_1.00u
- K16: value 3 -> Super; footprint Switch_Keyboard_Cherry_MX:SW_Cherry_MX_PCB_1.00u -> PCM_Switch_Keyboard_Hotswap_Kailh:SW_Hotswap_Kailh_MX_1.00u
- K17: value End -> E; footprint Switch_Keyboard_Cherry_MX:SW_Cherry_MX_PCB_1.00u -> PCM_Switch_Keyboard_Hotswap_Kailh:SW_Hotswap_Kailh_MX_1.00u
- K18: value Esc -> D; footprint Switch_Keyboard_Cherry_MX:SW_Cherry_MX_PCB_1.00u -> PCM_Switch_Keyboard_Hotswap_Kailh:SW_Hotswap_Kailh_MX_1.00u
- K19: value A -> C; footprint Switch_Keyboard_Cherry_MX:SW_Cherry_MX_PCB_1.00u -> PCM_Switch_Keyboard_Hotswap_Kailh:SW_Hotswap_Kailh_MX_1.00u
- K2: value Q -> End; footprint Switch_Keyboard_Cherry_MX:SW_Cherry_MX_PCB_1.00u -> PCM_Switch_Keyboard_Hotswap_Kailh:SW_Hotswap_Kailh_MX_1.00u
- K20: value S -> &dArr;; footprint Switch_Keyboard_Cherry_MX:SW_Cherry_MX_PCB_1.00u -> PCM_Switch_Keyboard_Hotswap_Kailh:SW_Hotswap_Kailh_MX_1.00u
- K21: value D -> R; footprint Switch_Keyboard_Cherry_MX:SW_Cherry_MX_PCB_1.00u -> PCM_Switch_Keyboard_Hotswap_Kailh:SW_Hotswap_Kailh_MX_1.00u
- K22, K45: footprint Switch_Keyboard_Cherry_MX:SW_Cherry_MX_PCB_1.00u -> PCM_Switch_Keyboard_Hotswap_Kailh:SW_Hotswap_Kailh_MX_1.00u
- K23: value G -> V; footprint Switch_Keyboard_Cherry_MX:SW_Cherry_MX_PCB_1.00u -> PCM_Switch_Keyboard_Hotswap_Kailh:SW_Hotswap_Kailh_MX_1.00u
- K24: value H -> T; footprint Switch_Keyboard_Cherry_MX:SW_Cherry_MX_PCB_1.00u -> PCM_Switch_Keyboard_Hotswap_Kailh:SW_Hotswap_Kailh_MX_1.00u
- K25: value J -> G; footprint Switch_Keyboard_Cherry_MX:SW_Cherry_MX_PCB_1.00u -> PCM_Switch_Keyboard_Hotswap_Kailh:SW_Hotswap_Kailh_MX_1.00u
- K26: value K -> B; footprint Switch_Keyboard_Cherry_MX:SW_Cherry_MX_PCB_1.00u -> PCM_Switch_Keyboard_Hotswap_Kailh:SW_Hotswap_Kailh_MX_1.00u
- K27: value L -> Blank; footprint Switch_Keyboard_Cherry_MX:SW_Cherry_MX_PCB_1.00u -> PCM_Switch_Keyboard_Hotswap_Kailh:SW_Hotswap_Kailh_MX_1.00u
- K28: value ; -> Y; footprint Switch_Keyboard_Cherry_MX:SW_Cherry_MX_PCB_1.00u -> PCM_Switch_Keyboard_Hotswap_Kailh:SW_Hotswap_Kailh_MX_1.00u
- K29: value ' -> H; footprint Switch_Keyboard_Cherry_MX:SW_Cherry_MX_PCB_1.00u -> PCM_Switch_Keyboard_Hotswap_Kailh:SW_Hotswap_Kailh_MX_1.00u
- K3: value W -> Vol +; footprint Switch_Keyboard_Cherry_MX:SW_Cherry_MX_PCB_1.00u -> PCM_Switch_Keyboard_Hotswap_Kailh:SW_Hotswap_Kailh_MX_1.00u
- K30: value Return -> N; footprint Switch_Keyboard_Cherry_MX:SW_Cherry_MX_PCB_1.00u -> PCM_Switch_Keyboard_Hotswap_Kailh:SW_Hotswap_Kailh_MX_1.00u
- K31: value 4 -> U; footprint Switch_Keyboard_Cherry_MX:SW_Cherry_MX_PCB_1.00u -> PCM_Switch_Keyboard_Hotswap_Kailh:SW_Hotswap_Kailh_MX_1.00u
- K32: value 5 -> J; footprint Switch_Keyboard_Cherry_MX:SW_Cherry_MX_PCB_1.00u -> PCM_Switch_Keyboard_Hotswap_Kailh:SW_Hotswap_Kailh_MX_1.00u
- K33: value 6 -> M; footprint Switch_Keyboard_Cherry_MX:SW_Cherry_MX_PCB_1.00u -> PCM_Switch_Keyboard_Hotswap_Kailh:SW_Hotswap_Kailh_MX_1.00u
- K34: value Vol + -> &uArr;; footprint Switch_Keyboard_Cherry_MX:SW_Cherry_MX_PCB_1.00u -> PCM_Switch_Keyboard_Hotswap_Kailh:SW_Hotswap_Kailh_MX_1.00u
- K35: value Shift -> I; footprint Switch_Keyboard_Cherry_MX:SW_Cherry_MX_PCB_1.00u -> PCM_Switch_Keyboard_Hotswap_Kailh:SW_Hotswap_Kailh_MX_1.00u
- K36: value Z -> K; footprint Switch_Keyboard_Cherry_MX:SW_Cherry_MX_PCB_1.00u -> PCM_Switch_Keyboard_Hotswap_Kailh:SW_Hotswap_Kailh_MX_1.00u
- K37: value X -> ,; footprint Switch_Keyboard_Cherry_MX:SW_Cherry_MX_PCB_1.00u -> PCM_Switch_Keyboard_Hotswap_Kailh:SW_Hotswap_Kailh_MX_1.00u
- K38: value C -> Alt; footprint Switch_Keyboard_Cherry_MX:SW_Cherry_MX_PCB_1.00u -> PCM_Switch_Keyboard_Hotswap_Kailh:SW_Hotswap_Kailh_MX_1.00u
- K39: value V -> O; footprint Switch_Keyboard_Cherry_MX:SW_Cherry_MX_PCB_1.00u -> PCM_Switch_Keyboard_Hotswap_Kailh:SW_Hotswap_Kailh_MX_1.00u
- K4: value E -> Vol -; footprint Switch_Keyboard_Cherry_MX:SW_Cherry_MX_PCB_1.00u -> PCM_Switch_Keyboard_Hotswap_Kailh:SW_Hotswap_Kailh_MX_1.00u
- K40: value B -> L; footprint Switch_Keyboard_Cherry_MX:SW_Cherry_MX_PCB_1.00u -> PCM_Switch_Keyboard_Hotswap_Kailh:SW_Hotswap_Kailh_MX_1.00u
- K41: value N -> .; footprint Switch_Keyboard_Cherry_MX:SW_Cherry_MX_PCB_1.00u -> PCM_Switch_Keyboard_Hotswap_Kailh:SW_Hotswap_Kailh_MX_1.00u
- K42: value M -> Fn; footprint Switch_Keyboard_Cherry_MX:SW_Cherry_MX_PCB_1.00u -> PCM_Switch_Keyboard_Hotswap_Kailh:SW_Hotswap_Kailh_MX_1.00u
- K43: value , -> P; footprint Switch_Keyboard_Cherry_MX:SW_Cherry_MX_PCB_1.00u -> PCM_Switch_Keyboard_Hotswap_Kailh:SW_Hotswap_Kailh_MX_1.00u
- K44: value . -> ;; footprint Switch_Keyboard_Cherry_MX:SW_Cherry_MX_PCB_1.00u -> PCM_Switch_Keyboard_Hotswap_Kailh:SW_Hotswap_Kailh_MX_1.00u
- K46: value Shift -> Back Space; footprint Switch_Keyboard_Cherry_MX:SW_Cherry_MX_PCB_1.00u -> PCM_Switch_Keyboard_Hotswap_Kailh:SW_Hotswap_Kailh_MX_1.00u
- K47: value 7 -> '; footprint Switch_Keyboard_Cherry_MX:SW_Cherry_MX_PCB_1.00u -> PCM_Switch_Keyboard_Hotswap_Kailh:SW_Hotswap_Kailh_MX_1.00u
- K48: value 8 -> Shift; footprint Switch_Keyboard_Cherry_MX:SW_Cherry_MX_PCB_1.00u -> PCM_Switch_Keyboard_Hotswap_Kailh:SW_Hotswap_Kailh_MX_1.00u
- K49: value 9 -> &larr;; footprint Switch_Keyboard_Cherry_MX:SW_Cherry_MX_PCB_1.00u -> PCM_Switch_Keyboard_Hotswap_Kailh:SW_Hotswap_Kailh_MX_1.00u
- K5: value R -> Tab; footprint Switch_Keyboard_Cherry_MX:SW_Cherry_MX_PCB_1.00u -> PCM_Switch_Keyboard_Hotswap_Kailh:SW_Hotswap_Kailh_MX_1.00u
- K50: value &uarr; -> Delete; footprint Switch_Keyboard_Cherry_MX:SW_Cherry_MX_PCB_1.00u -> PCM_Switch_Keyboard_Hotswap_Kailh:SW_Hotswap_Kailh_MX_1.00u
- K51: value Vol - -> Return; footprint Switch_Keyboard_Cherry_MX:SW_Cherry_MX_PCB_1.00u -> PCM_Switch_Keyboard_Hotswap_Kailh:SW_Hotswap_Kailh_MX_1.00u
- K52: value Ctrl -> &uarr;; footprint Switch_Keyboard_Cherry_MX:SW_Cherry_MX_PCB_1.25u -> PCM_Switch_Keyboard_Hotswap_Kailh:SW_Hotswap_Kailh_MX_1.00u
- K53: value Alt -> &darr;; footprint Switch_Keyboard_Cherry_MX:SW_Cherry_MX_PCB_1.25u -> PCM_Switch_Keyboard_Hotswap_Kailh:SW_Hotswap_Kailh_MX_1.00u
- K54: value Super -> &rarr;; footprint Switch_Keyboard_Cherry_MX:SW_Cherry_MX_PCB_1.25u -> PCM_Switch_Keyboard_Hotswap_Kailh:SW_Hotswap_Kailh_MX_1.00u
- K55: value &dArr; -> 1; footprint Switch_Keyboard_Cherry_MX:SW_Cherry_MX_PCB_1.25u -> PCM_Switch_Keyboard_Hotswap_Kailh:SW_Hotswap_Kailh_MX_1.00u
- K56: value Blank -> 4; footprint Switch_Keyboard_Cherry_MX:SW_Cherry_MX_PCB_2.00u -> PCM_Switch_Keyboard_Hotswap_Kailh:SW_Hotswap_Kailh_MX_1.00u
- K57: value &uArr; -> 7; footprint Switch_Keyboard_Cherry_MX:SW_Cherry_MX_PCB_1.25u -> PCM_Switch_Keyboard_Hotswap_Kailh:SW_Hotswap_Kailh_MX_1.00u
- K58: value Alt -> 2; footprint Switch_Keyboard_Cherry_MX:SW_Cherry_MX_PCB_1.25u -> PCM_Switch_Keyboard_Hotswap_Kailh:SW_Hotswap_Kailh_MX_1.00u
- K59: value Fn -> 5; footprint Switch_Keyboard_Cherry_MX:SW_Cherry_MX_PCB_1.25u -> PCM_Switch_Keyboard_Hotswap_Kailh:SW_Hotswap_Kailh_MX_1.00u
- K6: value T -> Esc; footprint Switch_Keyboard_Cherry_MX:SW_Cherry_MX_PCB_1.00u -> PCM_Switch_Keyboard_Hotswap_Kailh:SW_Hotswap_Kailh_MX_1.00u
- K60: value 0 -> 8; footprint Switch_Keyboard_Cherry_MX:SW_Cherry_MX_PCB_1.00u -> PCM_Switch_Keyboard_Hotswap_Kailh:SW_Hotswap_Kailh_MX_1.00u
- K61: value Enter -> 0; footprint Switch_Keyboard_Cherry_MX:SW_Cherry_MX_PCB_1.00u -> PCM_Switch_Keyboard_Hotswap_Kailh:SW_Hotswap_Kailh_MX_1.00u
- K62: value &larr; -> 3; footprint Switch_Keyboard_Cherry_MX:SW_Cherry_MX_PCB_1.00u -> PCM_Switch_Keyboard_Hotswap_Kailh:SW_Hotswap_Kailh_MX_1.00u
- K63: value &darr; -> 6; footprint Switch_Keyboard_Cherry_MX:SW_Cherry_MX_PCB_1.00u -> PCM_Switch_Keyboard_Hotswap_Kailh:SW_Hotswap_Kailh_MX_1.00u
- K64: value &rarr; -> 9; footprint Switch_Keyboard_Cherry_MX:SW_Cherry_MX_PCB_1.00u -> PCM_Switch_Keyboard_Hotswap_Kailh:SW_Hotswap_Kailh_MX_1.00u
- K7: value Y -> Shift; footprint Switch_Keyboard_Cherry_MX:SW_Cherry_MX_PCB_1.00u -> PCM_Switch_Keyboard_Hotswap_Kailh:SW_Hotswap_Kailh_MX_1.00u
- K8: value U -> Ctrl; footprint Switch_Keyboard_Cherry_MX:SW_Cherry_MX_PCB_1.00u -> PCM_Switch_Keyboard_Hotswap_Kailh:SW_Hotswap_Kailh_MX_1.00u
- K9: value I -> Q; footprint Switch_Keyboard_Cherry_MX:SW_Cherry_MX_PCB_1.00u -> PCM_Switch_Keyboard_Hotswap_Kailh:SW_Hotswap_Kailh_MX_1.00u
- U1: value Pico -> USBLC6-2SC6; footprint MCU_RaspberryPi_and_Boards:RPi_Pico_SMD_TH -> Package_TO_SOT_SMD:SOT-23-6
- moved U1 242.7 mm to (318.1, 89.2), turned to 0 degrees
- moved C1 72.7 mm to (341.1, 39.3)
- moved C2 63.5 mm to (341.3, 44.0)
- moved D_RGB9 12.5 mm to (202.2, 96.2)
- moved D_RGB12 11.3 mm to (181.7, 96.7)
- moved D13 7.25 mm to (300.8, 94.0)
Connections:
- C1 pad 1: VCC -> VBUS
- C2 pad 1: VCC -> +3V3
- D10 pad 1: /Row_0 -> /Row_1
- D11 pad 1: /Row_0 -> /Row_2
- D12 pad 1: /Row_0 -> /Row_3
- D14 pad 1: /Row_0 -> /Row_1
- D15 pad 1: /Row_0 -> /Row_2
- D16 pad 1: /Row_0 -> /Row_3
- D17 pad 1: /Row_1 -> /Row_0
- D19 pad 1: /Row_1 -> /Row_2
- D2 pad 1: /Row_0 -> /Row_1
- D20 pad 1: /Row_1 -> /Row_3
- D21 pad 1: /Row_1 -> /Row_0
- D23 pad 1: /Row_1 -> /Row_2
- D24 pad 1: /Row_1 -> /Row_0
- D26 pad 1: /Row_1 -> /Row_2
- D27 pad 1: /Row_1 -> /Row_3
- D28 pad 1: /Row_1 -> /Row_0
- D3 pad 1: /Row_0 -> /Row_2
- D30 pad 1: /Row_1 -> /Row_2
- D31 pad 1: /Row_1 -> /Row_0
- D33 pad 1: /Row_1 -> /Row_2
- D34 pad 1: /Row_2 -> /Row_3
- D35 pad 1: /Row_2 -> /Row_0
- D36 pad 1: /Row_2 -> /Row_1
- D38 pad 1: /Row_2 -> /Row_3
- D39 pad 1: /Row_2 -> /Row_0
- D4 pad 1: /Row_0 -> /Row_3
- D40 pad 1: /Row_2 -> /Row_1
- D42 pad 1: /Row_2 -> /Row_3
- D43 pad 1: /Row_2 -> /Row_0
- D44 pad 1: /Row_2 -> /Row_1
- D46 pad 1: /Row_2 -> /Row_0
- D47 pad 1: /Row_2 -> /Row_1
- D49 pad 1: /Row_2 -> /Row_3
- D50 pad 1: /Row_2 -> /Row_0
- D51 pad 1: /Row_3 -> /Row_1
- D52 pad 1: /Row_3 -> /Row_2
- D55 pad 1: /Row_3 -> /Row_0
- D56 pad 1: /Row_3 -> /Row_1
- D57 pad 1: /Row_3 -> /Row_2
- D58 pad 1: /Row_3 -> /Row_0
- D59 pad 1: /Row_3 -> /Row_1
- D6 pad 1: /Row_0 -> /Row_1
- D60 pad 1: /Row_3 -> /Row_2
- D62 pad 1: /Row_3 -> /Row_0
- D63 pad 1: /Row_3 -> /Row_1
- D64 pad 1: /Row_3 -> /Row_2
- D7 pad 1: /Row_0 -> /Row_2
- D8 pad 1: /Row_0 -> /Row_3
- D_RGB1 pad 1: VCC -> VBUS
- D_RGB1 pad 2: Net-(D_RGB1-Pad2) -> Net-(D_RGB1-DOUT)
- D_RGB1 pad 4: Net-(D_RGB1-Pad4) -> /LEDs/D_IN
- D_RGB10 pad 1: VCC -> VBUS
- D_RGB10 pad 2: Net-(D_RGB10-Pad2) -> Net-(D_RGB10-DOUT)
- D_RGB10 pad 4: Net-(D_RGB10-Pad4) -> Net-(D_RGB10-DIN)
- D_RGB11 pad 1: VCC -> VBUS
- D_RGB11 pad 2: Net-(D_RGB11-Pad2) -> Net-(D_RGB11-DOUT)
- D_RGB11 pad 4: Net-(D_RGB10-Pad2) -> Net-(D_RGB11-DIN)
- D_RGB12 pad 1: VCC -> VBUS
- D_RGB12 pad 2: Net-(D_RGB12-Pad2) -> Net-(D_RGB12-DOUT)
- D_RGB12 pad 4: Net-(D_RGB11-Pad2) -> Net-(D_RGB10-DOUT)
- D_RGB13 pad 1: VCC -> VBUS
- D_RGB13 pad 2: unconnected-(D_RGB13-Pad2) -> Net-(D_RGB13-DOUT)
- D_RGB13 pad 4: Net-(D_RGB12-Pad2) -> Net-(D_RGB11-DOUT)
- D_RGB2 pad 1: VCC -> VBUS
- D_RGB2 pad 2: Net-(D_RGB2-Pad2) -> Net-(D_RGB2-DOUT)
- D_RGB2 pad 4: Net-(D_RGB1-Pad2) -> Net-(D_RGB12-DOUT)
- D_RGB3 pad 1: VCC -> VBUS
- D_RGB3 pad 2: Net-(D_RGB3-Pad2) -> Net-(D_RGB3-DOUT)
- D_RGB3 pad 4: Net-(D_RGB2-Pad2) -> Net-(D_RGB13-DOUT)
- D_RGB4 pad 1: VCC -> VBUS
- D_RGB4 pad 2: Net-(D_RGB5-Pad4) -> Net-(D_RGB4-DOUT)
- D_RGB4 pad 4: Net-(D_RGB3-Pad2) -> Net-(D_RGB1-DOUT)
- D_RGB5 pad 1: VCC -> VBUS
- D_RGB5 pad 2: Net-(D_RGB5-Pad2) -> unconnected-(D_RGB5-DOUT-Pad2)
- D_RGB5 pad 4: Net-(D_RGB5-Pad4) -> Net-(D_RGB2-DOUT)
- D_RGB6 pad 1: VCC -> VBUS
- D_RGB6 pad 2: Net-(D_RGB6-Pad2) -> Net-(D_RGB6-DOUT)
- D_RGB6 pad 4: Net-(D_RGB5-Pad2) -> Net-(D_RGB3-DOUT)
- D_RGB7 pad 1: VCC -> VBUS
- D_RGB7 pad 2: Net-(D_RGB7-Pad2) -> Net-(D_RGB7-DOUT)
- D_RGB7 pad 4: Net-(D_RGB6-Pad2) -> Net-(D_RGB4-DOUT)
- D_RGB8 pad 1: VCC -> VBUS
- D_RGB8 pad 2: Net-(D_RGB8-Pad2) -> Net-(D_RGB10-DIN)
- D_RGB8 pad 4: Net-(D_RGB7-Pad2) -> Net-(D_RGB6-DOUT)
- D_RGB9 pad 1: VCC -> VBUS
- D_RGB9 pad 2: Net-(D_RGB10-Pad4) -> Net-(D_RGB11-DIN)
- D_RGB9 pad 4: Net-(D_RGB8-Pad2) -> Net-(D_RGB7-DOUT)
- K1 pad 1: /Col_1 -> /Col_0
- K10 pad 1: /Col_10 -> /Col_2
- K11 pad 1: /Col_11 -> /Col_2
- K12 pad 1: /Col_12 -> /Col_2
- K13 pad 1: /Col_13 -> /Col_3
- K14 pad 1: /Col_14 -> /Col_3
- K15 pad 1: /Col_15 -> /Col_3
- K16 pad 1: /Col_16 -> /Col_4
- K17 pad 1: /Col_0 -> /Col_4
- K18 pad 1: /Col_1 -> /Col_4
- K19 pad 1: /Col_2 -> /Col_4
- K2 pad 1: /Col_2 -> /Col_0
- K20 pad 1: /Col_3 -> /Col_5
- K21 pad 1: /Col_4 -> /Col_5
- K23 pad 1: /Col_6 -> /Col_5
- K24 pad 1: /Col_7 -> /Col_6
- K25 pad 1: /Col_8 -> /Col_6
- K26 pad 1: /Col_9 -> /Col_6
- K27 pad 1: /Col_10 -> /Col_6
- K28 pad 1: /Col_11 -> /Col_7
- K29 pad 1: /Col_12 -> /Col_7
- K3 pad 1: /Col_3 -> /Col_0
- K30 pad 1: /Col_13 -> /Col_7
- K31 pad 1: /Col_14 -> /Col_8
- K32 pad 1: /Col_15 -> /Col_8
- K33 pad 1: /Col_16 -> /Col_8
- K34 pad 1: /Col_0 -> /Col_8
- K35 pad 1: /Col_1 -> /Col_9
- K36 pad 1: /Col_2 -> /Col_9
- K37 pad 1: /Col_3 -> /Col_9
- K38 pad 1: /Col_4 -> /Col_9
- K39 pad 1: /Col_5 -> /Col_10
- K4 pad 1: /Col_4 -> /Col_0
- K40 pad 1: /Col_6 -> /Col_10
- K41 pad 1: /Col_7 -> /Col_10
- K42 pad 1: /Col_8 -> /Col_10
- K43 pad 1: /Col_9 -> /Col_11
- K44 pad 1: /Col_10 -> /Col_11
- K47 pad 1: /Col_14 -> /Col_12
- K48 pad 1: /Col_15 -> /Col_12
- K49 pad 1: /Col_16 -> /Col_12
- K5 pad 1: /Col_5 -> /Col_1
- K51 pad 1: /Col_0 -> /Col_13
- K52 pad 1: /Col_1 -> /Col_13
- K53 pad 1: /Col_2 -> /Col_13
- K54 pad 1: /Col_4 -> /Col_14
- K55 pad 1: /Col_5 -> /Col_14
- K56 pad 1: /Col_6 -> /Col_14
- K57 pad 1: /Col_8 -> /Col_14
- K58 pad 1: /Col_9 -> /Col_15
- K59 pad 1: /Col_10 -> /Col_15
- K6 pad 1: /Col_6 -> /Col_1
- K61 pad 1: /Col_16 -> /Col_15
- K62 pad 1: /Col_12 -> /Col_16
- K63 pad 1: /Col_13 -> /Col_16
- K64 pad 1: /Col_14 -> /Col_16
- K7 pad 1: /Col_7 -> /Col_1
- K8 pad 1: /Col_8 -> /Col_1
- K9 pad 1: /Col_9 -> /Col_2
- U1 pad 1: /Col_0 -> /USB/D-
- U1 pad 2: /Col_1 -> GND
- U1 pad 3: GND -> /USB/D+
- U1 pad 4: /Col_2 -> /USB_D+
- U1 pad 5: /Col_15 -> VBUS
- U1 pad 6: /Col_14 -> /USB_D-
Routing:
- net /Row_0: track 371.4 -> 0.00 mm
- net /Row_1: track 371.1 -> 0.00 mm, vias 2 -> 0
- net /Col_16: track 360.4 -> 0.00 mm
- net /Row_3: track 353.6 -> 0.00 mm
- net /Row_2: track 341.4 -> 0.00 mm
- net /Col_15: track 324.8 -> 0.00 mm
- net /Col_13: track 314.9 -> 0.00 mm
- net /Col_14: track 310.1 -> 0.00 mm
- net /Col_12: track 263.6 -> 0.00 mm
- net Net-(D_RGB1-Pad4): track 247.6 -> 0.00 mm, vias 1 -> 0
- net /Col_10: track 227.1 -> 0.00 mm
- net Net-(D_RGB1-Pad2): track 222.5 -> 0.00 mm, vias 2 -> 0
- net /Col_11: track 221.7 -> 0.00 mm
- net /Col_9: track 206.1 -> 0.00 mm
- net Net-(D_RGB12-Pad2): track 194.0 -> 0.00 mm, vias 6 -> 0
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- added copper zone on B.Cu, net GND
- removed copper zone on B.Cu, net VCC
Other:
- board size 340.4 x 81.3 mm -> 336.5 x 81.2 mm
- rule pad_to_mask_clearance: 0 -> 0.051
