File: Mimic40_plate.kicad_pcb (KiCad board)
At the start: 2 copper layers, 313.8 x 81.2 mm, 70 parts, among them K1 Home, K10 I, K11 O, K12 P, K13 Back Space, K14 Delete, K15 1, K16 2, K18 End, K19 Esc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

Commit message: finishing touches b4 prod
Parts:
- K56: footprint kbd:1u_plate -> kbd:2u_plate_stab
- turned K56 to 0 degrees
