File: LEDs.kicad_sch (KiCad schematic)
At the start: 66 parts, among them J5 Case Lighting

Commit message: usb changes for high power (leds)
Parts:
- added C10, C11, C12, C13, C14, C15, C16, C17, C19, C2, C20, C21, C22, C23, C24, C25, C26, C27, C28, C29, C3, C30, C31, C32, C33, C34, C35, C36, C37, C38, C39, C4, C40, C41, C42, C43, C44, C45, C46, C47, C48, C49, C5, C50, C52, C53, C54, C55, C6, C61, C62, C64, C65, C66, C67, C68, C69, C7, C70, C8, C9: 100n, Capacitor_SMD:C_0402_1005Metric, symbol Device:C
- added R1, R8: 500, Resistor_SMD:R_0402_1005Metric, symbol Device:R
- renumbered D_RGB16 to D_RGB1, D_RGB7 to D_RGB10, D_RGB6 to D_RGB11, D_RGB5 to D_RGB12, D_RGB4 to D_RGB13, D_RGB3 to D_RGB14, D_RGB2 to D_RGB15, D_RGB1 to D_RGB16, D_RGB15 to D_RGB2, D_RGB14 to D_RGB3, D_RGB48 to D_RGB33, D_RGB47 to D_RGB34, D_RGB46 to D_RGB35, D_RGB44 to D_RGB36, D_RGB43 to D_RGB37, D_RGB42 to D_RGB38, D_RGB41 to D_RGB39, D_RGB13 to D_RGB4, D_RGB39 to D_RGB41, D_RGB38 to D_RGB42, D_RGB37 to D_RGB43, D_RGB36 to D_RGB44, D_RGB35 to D_RGB45, D_RGB34 to D_RGB46, D_RGB33 to D_RGB47, D_RGB45 to D_RGB48, D_RGB12 to D_RGB5, D_RGB54 to D_RGB51, D_RGB55 to D_RGB52, D_RGB56 to D_RGB53, D_RGB57 to D_RGB54, D_RGB58 to D_RGB55, D_RGB59 to D_RGB56, D_RGB60 to D_RGB57, D_RGB61 to D_RGB58, D_RGB51 to D_RGB59, D_RGB11 to D_RGB6, D_RGB52 to D_RGB60, D_RGB53 to D_RGB61, D_RGB10 to D_RGB7, D_RGB9 to D_RGB8, D_RGB8 to D_RGB9, J5 to J4, JP1 to JP4, JP6 to JP5, JP8 to JP9
Connections:
- net D_IN: now also R1.2; no longer D_RGB16.4 (DIN)
- net D_OUT: now also R8.1; no longer D_RGB58.2 (DOUT)
- net GND: now also C10.2, C11.2, C12.2, C13.2, C14.2, C15.2, C16.2, C17.2, C19.2, C2.2, C20.2, C21.2, C22.2, C23.2, C24.2, C25.2, C26.2, C27.2, C28.2, C29.2, C3.2, C30.2, C31.2, C32.2, C33.2, C34.2, C35.2, C36.2, C37.2, C38.2, C39.2, C4.2, C40.2, C41.2, C42.2, C43.2, C44.2, C45.2, C46.2, C47.2, C48.2, C49.2, C5.2, C50.2, C52.2, C53.2, C54.2, C55.2, C6.2, C61.2, C62.2, C64.2, C65.2, C66.2, C67.2, C68.2, C69.2, C7.2, C70.2, C8.2, C9.2
- net VBUS: now also C10.1, C11.1, C12.1, C13.1, C14.1, C15.1, C16.1, C17.1, C19.1, C2.1, C20.1, C21.1, C22.1, C23.1, C24.1, C25.1, C26.1, C27.1, C28.1, C29.1, C3.1, C30.1, C31.1, C32.1, C33.1, C34.1, C35.1, C36.1, C37.1, C38.1, C39.1, C4.1, C40.1, C41.1, C42.1, C43.1, C44.1, C45.1, C46.1, C47.1, C48.1, C49.1, C5.1, C50.1, C52.1, C53.1, C54.1, C55.1, C6.1, C61.1, C62.1, C64.1, C65.1, C66.1, C67.1, C68.1, C69.1, C7.1, C70.1, C8.1, C9.1
- net D_{in}_{k}: now reaches D_RGB6.4 (DIN), D_RGB7.2 (DOUT)
- net D_{in}_{j}: now reaches D_RGB1.4 (DIN), D_RGB2.2 (DOUT)
- net D_{in}_{b}: now reaches D_RGB59.4 (DIN), JP9.2 (B)
- net D_{in}_{h}: now reaches D_RGB25.2 (DOUT), D_RGB26.4 (DIN)
- net D_{in}_{g}: now reaches D_RGB30.2 (DOUT), D_RGB31.4 (DIN)
- net D_{in}_{a}: now reaches D_RGB52.2 (DOUT), D_RGB53.4 (DIN)
- net D_{in}_{f}: now reaches D_RGB44.4 (DIN), D_RGB45.2 (DOUT)
- net D_{in}_{i}: now reaches D_RGB20.2 (DOUT), D_RGB21.4 (DIN)
- net D_{in}_{l}: now reaches D_RGB11.4 (DIN), D_RGB12.2 (DOUT)
- net D_{in}_{e}: now reaches D_RGB39.4 (DIN), D_RGB40.2 (DOUT)
- net D_{in}_{c}: now reaches D_RGB35.4 (DIN), D_RGB48.2 (DOUT)
- new net: D_RGB16.4 (DIN), R1.1
- new net: D_RGB58.2 (DOUT), R8.2
- no-connect marks 1 -> 0
Other:
- title: (none) -> Per-key Addressable RGB
- moved on the sheet: D_RGB1, D_RGB10, D_RGB11, D_RGB12, D_RGB13, D_RGB14, D_RGB15, D_RGB16, D_RGB17, D_RGB18, D_RGB19, D_RGB2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

Commit message: bulk cap and level shifter (still need to lay out)
Parts:
- C10, C11, C12, C13, C14, C15, C16, C17, C19, C2, C20, C21, C22, C23, C24, C25, C26, C27, C28, C29, C3, C30, C31, C32, C33, C34, C35, C36, C37, C38, C39, C4, C40, C41, C42, C43, C44, C45, C46, C47, C48, C49, C5, C50, C52, C53, C54, C55, C6, C61, C62, C64, C65, C66, C67, C68, C69, C7, C70, C8, C9: value 100n -> 100nF; LCSC (none) -> C1525; MPN (none) -> CL05B104KO5NNNC; Manufacturer (none) -> Samsung Electro-Mechanics
- J4: MPN (none) -> DNP
- JP4, JP5, JP7, JP9: MPN (none) -> DNP; now not fitted
- R1, R8: LCSC (none) -> C17168; MPN (none) -> 0402WGF0000TCE; Manufacturer (none) -> UNIROYAL
Other:
- note added: "https://learn.adafruit.com/adafruit-neopixel-uberguide/powering-neopixels"
- note added: "https://learn.adafruit.com/led-tricks-gamma-correction"
- note added: "https://learn.adafruit.com/sipping-power-with-neopixels"
