File: LEDs.kicad_sch (KiCad schematic)
At the start: 129 parts, among them J4 Case Lighting

Commit message: bulk caps for power (todo, split 470uF cap so that it can be shorter)
Parts:
- added C81, C82, C83, C84, C85: 100uF, Capacitor_SMD:CP_Elec_6.3x4.5, symbol Device:C_Polarized
- J4: footprint Connector_PinHeader_2.54mm:PinHeader_1x04_P2.54mm_Vertical -> Connector_PinHeader_2.54mm:PinHeader_1x03_P2.54mm_Vertical; symbol Connector_Generic:Conn_02x02_Odd_Even -> Connector_Generic:Conn_01x03; now in the parts list
Connections:
- net D_IN: no longer J4.3 (Pin_3)
- net GND: now also C81.2, C82.2, C83.2, C84.2, C85.2
- net VBUS: now also J4.3 (Pin_3), C81.1, C82.1, C83.1, C84.1, C85.1; no longer J4.4 (Pin_4)
Other:
- note added: "bulk cap for power filtering"

Commit message: add debug led, make bulk caps smaller, export plate and bottom for rudimentary case
Parts:
- C81, C82, C83, C84, C85: footprint Capacitor_SMD:CP_Elec_6.3x4.5 -> Capacitor_SMD:C_1206_3216Metric; LCSC C22388021 -> C15008; MPN EFVM025ADA101M0654 -> CL31A107MQHNNNE; Manufacturer FOLLON -> Samsung Electro-Mechanics
- R1, R8: value 500 -> 470; LCSC C17168 -> C25117; MPN 0402WGF0000TCE -> 0402WGF4700TCE
Changed lines of the file:
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@@
 			)
 		)
-		(property "Value" "500"
+		(property "Value" "470"
 			(at 128.27 85.09 90)
 			(effects
@@
 			)
 		)
-		(property "LCSC" "C17168"
+		(property "LCSC" "C25117"
 			(at 128.27 78.74 0)
 			(effects
@@
 			)
 		)
-		(property "MPN" "0402WGF0000TCE"
+		(property "MPN" "0402WGF4700TCE"
 			(at 128.27 78.74 0)
 			(effects
@@
 			)
 		)
-		(property "Value" "500"
+		(property "Value" "470"
 			(at 292.1 523.24 90)
 			(effects
@@
 			)
 		)
-		(property "LCSC" "C17168"
+		(property "LCSC" "C25117"
 			(at 292.1 527.05 0)
 			(effects
@@
 			)
 		)
-		(property "MPN" "0402WGF0000TCE"
+		(property "MPN" "0402WGF4700TCE"
 			(at 292.1 527.05 0)
 			(effects
@@
 			)
 		)
-		(property "Footprint" "Capacitor_SMD:CP_Elec_6.3x4.5"
+		(property "Footprint" "Capacitor_SMD:C_1206_3216Metric"
 			(at 96.2152 406.4 0)
 			(effects
@@
 			)
 		)
-		(property "LCSC" "C22388021"
+		(property "LCSC" "C15008"
 			(at 95.25 402.59 0)
 			(effects
@@
 			)
 		)
-		(property "MPN" "EFVM025ADA101M0654"
+		(property "MPN" "CL31A107MQHNNNE"
 			(at 95.25 402.59 0)
 			(effects
@@
 			)
 		)
-		(property "Manufacturer" "FOLLON"
+		(property "Manufacturer" "Samsung Electro-Mechanics"
 			(at 95.25 402.59 0)
 			(effects
@@
 			)
 		)
-		(property "Footprint" "Capacitor_SMD:CP_Elec_6.3x4.5"
+		(property "Footprint" "Capacitor_SMD:C_1206_3216Metric"
 			(at 96.2152 326.39 0)
 			(effects
@@
 			)
 		)
-		(property "LCSC" "C22388021"
+		(property "LCSC" "C15008"
 			(at 95.25 322.58 0)
 			(effects
@@
 			)
 		)
-		(property "MPN" "EFVM025ADA101M0654"
+		(property "MPN" "CL31A107MQHNNNE"
 			(at 95.25 322.58 0)
 			(effects
@@
 			)
 		)
-		(property "Manufacturer" "FOLLON"
+		(property "Manufacturer" "Samsung Electro-Mechanics"
 			(at 95.25 322.58 0)
 			(effects
@@
 			)
 		)
-		(property "Footprint" "Capacitor_SMD:CP_Elec_6.3x4.5"
+		(property "Footprint" "Capacitor_SMD:C_1206_3216Metric"
 			(at 96.2152 245.11 0)
 			(effects
@@
 			)
 		)
-		(property "LCSC" "C22388021"
+		(property "LCSC" "C15008"
 			(at 95.25 241.3 0)
 			(effects
@@
 			)
 		)
-		(property "MPN" "EFVM025ADA101M0654"
+		(property "MPN" "CL31A107MQHNNNE"
 			(at 95.25 241.3 0)
 			(effects
@@
 			)
 		)
-		(property "Manufacturer" "FOLLON"
+		(property "Manufacturer" "Samsung Electro-Mechanics"
 			(at 95.25 241.3 0)
 			(effects
@@
 			)
 		)
-		(property "Footprint" "Capacitor_SMD:CP_Elec_6.3x4.5"
+		(property "Footprint" "Capacitor_SMD:C_1206_3216Metric"
 			(at 96.2152 163.83 0)
 			(effects
@@
 			)
 		)
-		(property "LCSC" "C22388021"
+		(property "LCSC" "C15008"
 			(at 95.25 160.02 0)
 			(effects
@@
 			)
 		)
-		(property "MPN" "EFVM025ADA101M0654"
+		(property "MPN" "CL31A107MQHNNNE"
 			(at 95.25 160.02 0)
 			(effects
@@
 			)
 		)
-		(property "Manufacturer" "FOLLON"
+		(property "Manufacturer" "Samsung Electro-Mechanics"
 			(at 95.25 160.02 0)
 			(effects
@@
 			)
 		)
-		(property "Footprint" "Capacitor_SMD:CP_Elec_6.3x4.5"
+		(property "Footprint" "Capacitor_SMD:C_1206_3216Metric"
 			(at 96.2152 487.68 0)
 			(effects
@@
 			)
 		)
-		(property "LCSC" "C22388021"
+		(property "LCSC" "C15008"
 			(at 95.25 483.87 0)
 			(effects
@@
 			)
 		)
-		(property "MPN" "EFVM025ADA101M0654"
+		(property "MPN" "CL31A107MQHNNNE"
 			(at 95.25 483.87 0)
 			(effects
@@
 			)
 		)
-		(property "Manufacturer" "FOLLON"
+		(property "Manufacturer" "Samsung Electro-Mechanics"
 			(at 95.25 483.87 0)
 			(effects

Commit message: enlarge mounting holes, custom rules
Parts:
- JP4, JP5, JP7, JP9: value Jumper_2_Bridged -> Jumper_2_Small_Bridged; symbol Jumper:Jumper_2_Bridged -> Jumper:Jumper_2_Small_Bridged; now in the parts list
Other:
- moved on the sheet: C10, C11, C12, C13, C14, C15, C16, C17, C19, C2, C20, C21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

Commit message: fab output changes (part choice updates)
Parts:
- C10, C11, C12, C13, C14, C15, C16, C17, C19, C2, C20, C21, C22, C23, C24, C25, C26, C27, C28, C29, C3, C30, C31, C32, C33, C34, C35, C36, C37, C38, C39, C4, C40, C41, C42, C43, C44, C45, C46, C47, C48, C49, C5, C50, C52, C53, C54, C55, C6, C61, C62, C64, C65, C66, C67, C68, C69, C7, C70, C8, C81, C82, C83, C84, C85, C9, R1, R8: Type (none) -> SMD
- J4: Type DNS -> THT
