File: Mimic40.kicad_sch (KiCad schematic)
At the start: 14 parts, among them J3 Conn_01x04, J5 Conn_01x03

Commit message: fab output changes (part choice updates)
Parts:
- D65, R14: Type (none) -> SMD
- J3, J5: Type DNS -> THT
Changed lines of the file:
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@@
+			)
+		)
+		(property "Type" "SMD"
+			(at 190.5 130.81 0)
+			(effects
+				(font
+					(size 1.27 1.27)
+				)
+				(hide yes)
 			)
 		)
@@
 			)
 		)
+		(property "Type" "SMD"
+			(at 179.07 138.43 0)
+			(effects
+				(font
+					(size 1.27 1.27)
+				)
+				(hide yes)
+			)
+		)
 		(pin "1"
 		)
@@
 			)
 		)
-		(property "Type" "DNS"
+		(property "Type" "THT"
 			(at 229.87 203.2 0)
 			(effects
@@
 			)
 		)
-		(property "Type" "DNS"
+		(property "Type" "THT"
 			(at 165.1 203.2 0)
 			(effects
