File: USB.kicad_sch (KiCad schematic)
At the start: 12 parts, among them J2 USB_C_Receptacle_USB2.0_16P, U1 AMS1117-3.3, U2 USBLC6-2SC6

Commit message: fab output changes (part choice updates)
Parts:
- C79, C80, C86, C87, F1: Type (none) -> SMD
Changed lines of the file:
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@@
+			)
+		)
+		(property "Type" "SMD"
+			(at 64.77 100.33 0)
+			(effects
+				(font
+					(size 1.27 1.27)
+				)
+				(hide yes)
 			)
 		)
@@
 			)
 		)
+		(property "Type" "SMD"
+			(at 165.1 83.82 0)
+			(effects
+				(font
+					(size 1.27 1.27)
+				)
+				(hide yes)
+			)
+		)
 		(pin "2"
 		)
@@
 			)
 		)
+		(property "Type" "SMD"
+			(at 77.47 100.33 0)
+			(effects
+				(font
+					(size 1.27 1.27)
+				)
+				(hide yes)
+			)
+		)
 		(pin "2"
 		)
@@
 			)
 		)
+		(property "Type" "SMD"
+			(at 52.07 100.33 0)
+			(effects
+				(font
+					(size 1.27 1.27)
+				)
+				(hide yes)
+			)
+		)
 		(pin "2"
 		)
@@
 			(at 90.17 100.33 0)
 			(effects
+				(font
+					(size 1.27 1.27)
+				)
+				(hide yes)
+			)
+		)
+		(property "Type" "SMD"
+			(at 90.17 100.33 0)
+			(effects
